File: FluidNC-BOB v1.1.kicad_pcb (KiCad board)
At the start: 2 copper layers, 167.6 x 96.5 mm, 46 parts, among them J1 X_Limit, J10 Z_stepdir, J11 spindle_pwm_dir, J12 Flood_Mist, J13 GND, J14 GND, J15 +5v, J16 +5v, J2 Y_Limit, J3 Hold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

Commit message: Add files via upload
Parts:
- U10: footprint Package_DIP:DIP-14_W7.62mm_Socket_LongPads -> Package_DIP:DIP-14_W7.62mm_Socket
- U8, U9: footprint Package_DIP:DIP-20_W7.62mm_Socket_LongPads -> Package_DIP:DIP-20_W7.62mm_Socket
- moved G*** 7.39 mm to (142.5, 126.8)
Routing:
- net GND: track 427.9 -> 431.7 mm
- net +3V3: track 150.9 -> 149.6 mm
- net Net-(U1-D32): track 19.9 -> 21.1 mm
- net Net-(U1-D33): track 13.1 -> 13.8 mm
- net Net-(U1-D35): track 27.0 -> 27.7 mm
- net Net-(R12-Pad1): track 37.8 -> 38.4 mm
- net Net-(R7-Pad1): track 34.6 -> 33.9 mm
