File: FluidNC-BOB v1.1.kicad_sch (KiCad schematic)
At the start: 45 parts, among them J1 X_Limit, J10 Z_stepdir, J11 spindle_pwm_dir, J12 Flood_Mist, J13 GND, J14 GND, J15 +5v, J16 +5v, J2 Y_Limit, J3 Hold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

Commit message: Add files via upload
Parts:
- U10: footprint Package_DIP:DIP-14_W7.62mm_Socket_LongPads -> Package_DIP:DIP-14_W7.62mm_Socket
- U8, U9: footprint Package_DIP:DIP-20_W7.62mm_Socket_LongPads -> Package_DIP:DIP-20_W7.62mm_Socket
Changed lines of the file:
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@@
       (effects (font (size 1.27 1.27)))
     )
-    (property "Footprint" "Package_DIP:DIP-20_W7.62mm_Socket_LongPads" (at 132.08 110.49 0)
+    (property "Footprint" "Package_DIP:DIP-20_W7.62mm_Socket" (at 132.08 110.49 0)
       (effects (font (size 1.27 1.27)) hide)
     )
@@
       (effects (font (size 1.27 1.27)))
     )
-    (property "Footprint" "Package_DIP:DIP-20_W7.62mm_Socket_LongPads" (at 132.08 154.94 0)
+    (property "Footprint" "Package_DIP:DIP-20_W7.62mm_Socket" (at 132.08 154.94 0)
       (effects (font (size 1.27 1.27)) hide)
     )
@@
       (effects (font (size 1.27 1.27)) (justify left))
     )
-    (property "Footprint" "Package_DIP:DIP-14_W7.62mm_Socket_LongPads" (at 40.64 36.83 0)
+    (property "Footprint" "Package_DIP:DIP-14_W7.62mm_Socket" (at 40.64 36.83 0)
       (effects (font (size 1.27 1.27)) hide)
     )
@@
       (effects (font (size 1.27 1.27)))
     )
-    (property "Footprint" "Package_DIP:DIP-14_W7.62mm_Socket_LongPads" (at 119.38 64.77 0)
+    (property "Footprint" "Package_DIP:DIP-14_W7.62mm_Socket" (at 119.38 64.77 0)
       (effects (font (size 1.27 1.27)) hide)
     )
@@
       (effects (font (size 1.27 1.27)))
     )
-    (property "Footprint" "Package_DIP:DIP-14_W7.62mm_Socket_LongPads" (at 134.62 68.58 0)
+    (property "Footprint" "Package_DIP:DIP-14_W7.62mm_Socket" (at 134.62 68.58 0)
       (effects (font (size 1.27 1.27)) hide)
     )
@@
       (effects (font (size 1.27 1.27)))
     )
-    (property "Footprint" "Package_DIP:DIP-14_W7.62mm_Socket_LongPads" (at 182.88 81.28 0)
+    (property "Footprint" "Package_DIP:DIP-14_W7.62mm_Socket" (at 182.88 81.28 0)
       (effects (font (size 1.27 1.27)) hide)
     )
@@
       (effects (font (size 1.27 1.27)))
     )
-    (property "Footprint" "Package_DIP:DIP-14_W7.62mm_Socket_LongPads" (at 149.86 72.39 0)
+    (property "Footprint" "Package_DIP:DIP-14_W7.62mm_Socket" (at 149.86 72.39 0)
       (effects (font (size 1.27 1.27)) hide)
     )
@@
       (effects (font (size 1.27 1.27)))
     )
-    (property "Footprint" "Package_DIP:DIP-14_W7.62mm_Socket_LongPads" (at 167.64 76.2 0)
+    (property "Footprint" "Package_DIP:DIP-14_W7.62mm_Socket" (at 167.64 76.2 0)
       (effects (font (size 1.27 1.27)) hide)
     )
@@
       (effects (font (size 1.27 1.27)))
     )
-    (property "Footprint" "Package_DIP:DIP-14_W7.62mm_Socket_LongPads" (at 104.14 60.96 0)
-      (effects (font (size 1.27 1.27)) hide)
-    )
+    (property "Footprint" "Package_DIP:DIP-14_W7.62mm_Socket" (at 104.14 60.96 0)
+      (effects (font (size 1.27 1.27)) hide)
+    )
